File: HW_design/Access_control/LedIndicator.sch (KiCad schematic (older format))
At the start: 4 parts

Commit message: pcb design
Parts:
- D2, D3: renamed from D?; footprint (none) -> Diode_SMD:D_1206_3216Metric
- R7, R8: renamed from R?; footprint (none) -> Resistor_SMD:R_0805_2012Metric
Changed lines of the file:
@@
 GPIO05
 $Comp
-L Device:R R?
+L Device:R R7
 U 1 1 604CCEB8
 P 1650 900
-F 0 "R?" V 1443 900 50  0000 C CNN
+F 0 "R7" V 1443 900 50  0000 C CNN
 F 1 "220" V 1534 900 50  0000 C CNN
-F 2 "" V 1580 900 50  0001 C CNN
+F 2 "Resistor_SMD:R_0805_2012Metric" V 1580 900 50  0001 C CNN
 F 3 "~" H 1650 900 50  0001 C CNN
 	1    1650 900
@@
 $EndComp
 $Comp
-L Device:LED D?
+L Device:LED D2
 U 1 1 604CD3A3
 P 1950 1100
-F 0 "D?" V 1989 982 50  0000 R CNN
+F 0 "D2" V 1989 982 50  0000 R CNN
 F 1 "LED" V 1898 982 50  0000 R CNN
-F 2 "" H 1950 1100 50  0001 C CNN
+F 2 "Diode_SMD:D_1206_3216Metric" H 1950 1100 50  0001 C CNN
 F 3 "~" H 1950 1100 50  0001 C CNN
 	1    1950 1100
@@
 	1950 900  1950 950
 $Comp
-L power:GND #PWR?
+L power:GND #PWR0116
 U 1 1 604CDD45
 P 1950 1250
-F 0 "#PWR?" H 1950 1000 50  0001 C CNN
+F 0 "#PWR0116" H 1950 1000 50  0001 C CNN
 F 1 "GND" H 1955 1077 50  0000 C CNN
 F 2 "" H 1950 1250 50  0001 C CNN
@@
 GPIO15
 $Comp
-L Device:R R?
+L Device:R R8
 U 1 1 604CE252
 P 1650 1700
-F 0 "R?" V 1443 1700 50  0000 C CNN
+F 0 "R8" V 1443 1700 50  0000 C CNN
 F 1 "220" V 1534 1700 50  0000 C CNN
-F 2 "" V 1580 1700 50  0001 C CNN
+F 2 "Resistor_SMD:R_0805_2012Metric" V 1580 1700 50  0001 C CNN
 F 3 "~" H 1650 1700 50  0001 C CNN
 	1    1650 1700
@@
 	1350 1700 1500 1700
 $Comp
-L Device:LED D?
+L Device:LED D3
 U 1 1 604CE6D4
 P 1950 2000
-F 0 "D?" V 1989 1882 50  0000 R CNN
+F 0 "D3" V 1989 1882 50  0000 R CNN
 F 1 "LED" V 1898 1882 50  0000 R CNN
-F 2 "" H 1950 2000 50  0001 C CNN
+F 2 "Diode_SMD:D_1206_3216Metric" H 1950 2000 50  0001 C CNN
 F 3 "~" H 1950 2000 50  0001 C CNN
 	1    1950 2000
@@
 	1950 1700 1950 1850
 $Comp
-L power:GND #PWR?
+L power:GND #PWR0117
 U 1 1 604CF024
 P 1950 2150
-F 0 "#PWR?" H 1950 1900 50  0001 C CNN
+F 0 "#PWR0117" H 1950 1900 50  0001 C CNN
 F 1 "GND" H 1955 1977 50  0000 C CNN
 F 2 "" H 1950 2150 50  0001 C CNN
