File: HW_design/Access_control/Regulator.sch (KiCad schematic (older format))
At the start: 3 parts

Commit message: pcb design
Parts:
- C3, C4: renamed from C?; footprint (none) -> Capacitor_SMD:C_1206_3216Metric
- gave numbers to parts that had none: 1
Changed lines of the file:
@@
 $EndDescr
 $Comp
-L Regulator_Linear:AMS1117-3.3 U?
+L Regulator_Linear:AMS1117-3.3 U4
 U 1 1 604D73D7
 P 3350 1050
-F 0 "U?" H 3350 1292 50  0000 C CNN
+F 0 "U4" H 3350 1292 50  0000 C CNN
 F 1 "AMS1117-3.3" H 3350 1201 50  0000 C CNN
 F 2 "Package_TO_SOT_SMD:SOT-223-3_TabPin2" H 3350 1250 50  0001 C CNN
@@
 $EndComp
 $Comp
-L power:GND #PWR?
+L power:GND #PWR0110
 U 1 1 604D894F
 P 3350 1350
-F 0 "#PWR?" H 3350 1100 50  0001 C CNN
+F 0 "#PWR0110" H 3350 1100 50  0001 C CNN
 F 1 "GND" H 3355 1177 50  0000 C CNN
 F 2 "" H 3350 1350 50  0001 C CNN
@@
 	3650 1050 3800 1050
 $Comp
-L Device:C C?
+L Device:C C3
 U 1 1 604D98E4
 P 2950 1450
-F 0 "C?" H 3065 1496 50  0000 L CNN
+F 0 "C3" H 3065 1496 50  0000 L CNN
 F 1 "10uF" H 3065 1405 50  0000 L CNN
-F 2 "" H 2988 1300 50  0001 C CNN
+F 2 "Capacitor_SMD:C_1206_3216Metric" H 2988 1300 50  0001 C CNN
 F 3 "~" H 2950 1450 50  0001 C CNN
 	1    2950 1450
@@
 $EndComp
 $Comp
-L Device:C C?
+L Device:C C4
 U 1 1 604D9F4A
 P 3800 1450
-F 0 "C?" H 3915 1496 50  0000 L CNN
+F 0 "C4" H 3915 1496 50  0000 L CNN
 F 1 "10uF" H 3915 1405 50  0000 L CNN
-F 2 "" H 3838 1300 50  0001 C CNN
+F 2 "Capacitor_SMD:C_1206_3216Metric" H 3838 1300 50  0001 C CNN
 F 3 "~" H 3800 1450 50  0001 C CNN
 	1    3800 1450
@@
 	2950 1050 2950 1300
 $Comp
-L power:GND #PWR?
+L power:GND #PWR0111
 U 1 1 604DAF37
 P 2950 1700
-F 0 "#PWR?" H 2950 1450 50  0001 C CNN
+F 0 "#PWR0111" H 2950 1450 50  0001 C CNN
 F 1 "GND" H 2955 1527 50  0000 C CNN
 F 2 "" H 2950 1700 50  0001 C CNN
@@
 $EndComp
 $Comp
-L power:GND #PWR?
+L power:GND #PWR0112
 U 1 1 604DB2C5
 P 3800 1700
-F 0 "#PWR?" H 3800 1450 50  0001 C CNN
+F 0 "#PWR0112" H 3800 1450 50  0001 C CNN
 F 1 "GND" H 3805 1527 50  0000 C CNN
 F 2 "" H 3800 1700 50  0001 C CNN
