File: HW_design/Access_control/Access_control.kicad_pcb (KiCad board)
At the start: 2 copper layers, 30 parts, among them J1 Conn_01x08_Male, J2 Conn_01x02_Male, J3 NC, J4 RX, J5 TX, J6 Vcc, J7 NC, J8 GND, J9 Conn_01x02_Male, Q1 MMBT3904, U1 ESP-12E, U2 Bornera2, U3 Bornera2, U4 AMS1117-3.3

Commit message: fix pcb
Routing:
- net Vcc: track 157.2 -> 142.6 mm, vias 1 -> 2
Changed lines of the file:
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@@
     (thickness 1.6)
     (drawings 4)
-    (tracks 352)
+    (tracks 353)
     (zones 0)
     (modules 30)
@@
   (segment (start 150.9685 98.1075) (end 152.8695 98.1075) (width 0.3) (layer B.Cu) (net 3))
   (segment (start 149.8745 99.2015) (end 150.9685 98.1075) (width 0.3) (layer B.Cu) (net 3))
-  (segment (start 130.96649 95.30299) (end 132.0165 96.353) (width 0.3) (layer B.Cu) (net 3))
-  (segment (start 130.96649 72.80501) (end 130.96649 95.30299) (width 0.3) (layer B.Cu) (net 3))
-  (segment (start 135.0645 68.707) (end 130.96649 72.80501) (width 0.3) (layer B.Cu) (net 3))
-  (segment (start 137.795 68.707) (end 135.0645 68.707) (width 0.3) (layer B.Cu) (net 3))
-  (segment (start 138.43 69.342) (end 137.795 68.707) (width 0.3) (layer B.Cu) (net 3))
-  (segment (start 138.43 74.1045) (end 138.43 69.342) (width 0.3) (layer B.Cu) (net 3))
-  (segment (start 136.4615 76.073) (end 138.43 74.1045) (width 0.3) (layer B.Cu) (net 3))
   (segment (start 164.725499 81.873501) (end 164.725499 77.844501) (width 0.3) (layer B.Cu) (net 3))
   (segment (start 159.7085 86.8905) (end 164.725499 81.873501) (width 0.3) (layer B.Cu) (net 3))
@@
   (segment (start 134.62 96.821) (end 135.1915 96.2495) (width 0.3) (layer B.Cu) (net 3))
   (segment (start 134.62 98.806) (end 134.62 96.821) (width 0.3) (layer B.Cu) (net 3))
+  (segment (start 130.96649 95.30299) (end 132.0165 96.353) (width 0.3) (layer B.Cu) (net 3))
+  (segment (start 130.96649 95.30299) (end 130.10099 95.30299) (width 0.3) (layer B.Cu) (net 3))
+  (segment (start 130.10099 95.30299) (end 129.794 94.996) (width 0.3) (layer B.Cu) (net 3))
+  (via (at 132.842 76.581) (size 0.8) (drill 0.4) (layers F.Cu B.Cu) (net 3))
+  (segment (start 129.794 79.629) (end 132.842 76.581) (width 0.3) (layer B.Cu) (net 3))
+  (segment (start 129.794 94.996) (end 129.794 79.629) (width 0.3) (layer B.Cu) (net 3))
+  (segment (start 133.35 76.073) (end 136.4615 76.073) (width 0.3) (layer F.Cu) (net 3))
+  (segment (start 132.842 76.581) (end 133.35 76.073) (width 0.3) (layer F.Cu) (net 3))
   (segment (start 152.6295 95.5675) (end 152.8695 95.8075) (width 0.3) (layer B.Cu) (net 4))
   (segment (start 149.8745 95.5675) (end 152.6295 95.5675) (width 0.3) (layer B.Cu) (net 4))

Commit message: .
Other:
- board outline added: 44.4 x 66.3 mm
