File: HW_design/Access_control/Access_control.sch (KiCad schematic (older format))
At the start: 3 parts

Commit message: Schematic update
Parts:
- removed J?: Conn_01x08_Male, symbol Connector:Conn_01x08_Male
- added C?: 100nF, symbol Device:C
- added R? (x5): 12k, symbol Device:R
- added U? (x2): Bornera2, symbol Terminal:Bornera2
- C?: value C -> 100uF
Connections:
- net +3V3: now also R?.1, R?.1, R?.1, R?.1
- net GND: now also C?.2, R?.1, U?.2 (-), U?.2 (-)
- net RST: now reaches U?.1 (REST)
- net RST: now also C?.1, R?.2
- net GPIO15: now reaches U?.10 (GPIO15)
- net GPIO15: now also R?.2
- net GPIO02: now reaches U?.11 (GPIO2)
- net GPIO02: now also R?.2
- net GPIO00: now reaches U?.12 (GPIO0)
- net GPIO00: now also R?.2
- net GPIO04: now reaches U?.13 (GPIO4)
- net GPIO05: now reaches U?.14 (GPIO5)
- net RXD: now reaches U?.15 (RXD)
- net TXD: now reaches U?.16 (TXD)
- net MISO: now reaches U?.18 (MISO)
- net GPIO09: now reaches U?.19 (GPIO9)
- net GPIO10: now reaches U?.20 (GPIO10)
- net MOSI: now reaches U?.21 (MOSI)
- net SCL: now reaches U?.22 (SCLK)
- net EN: now reaches U?.3 (CH_PD)
- net EN: now also R?.2
- net GPIO16: now reaches U?.4 (GPIO16)
- net GPIO14: now reaches U?.5 (GPIO14)
- net GPIO12: now reaches U?.6 (GPIO12)
- net GPIO13: now reaches U?.7 (GPIO13)
- new net +12V: U?.1 (+)
- new net Rel_1_out: U?.1 (+)
- no-connect marks 0 -> 2
Other:
- note added: "1.0"
- note added: "ACCESS CONTROL"
- note added: "FTDI"
- note added: "Led indicators"
- note added: "Output"
- note added: "Power supply"
- note added: "Regulator"
- note added: "Relay"
- moved on the sheet: C?, U?

Commit message: pcb design
Parts:
- C1, C2: renamed from C?; footprint (none) -> Capacitor_SMD:C_1206_3216Metric
- R1, R2, R3, R4: renamed from R?; value 12k -> 10k; footprint (none) -> Resistor_SMD:R_0805_2012Metric
- R5: renamed from R?; footprint (none) -> Resistor_SMD:R_0805_2012Metric
- U1: renamed from U?; footprint (none) -> RF_Module:ESP-12E
- U2, U3: renamed from U?; footprint (none) -> Borneras:Bronera_2
Changed lines of the file:
@@
 Comment4 ""
 $EndDescr
-$Comp
-L ESP_8366_CUSTOM:ESP-12E U?
-U 1 1 60363FD8
-P 2100 1500
-F 0 "U?" H 2100 2265 50  0000 C CNN
-F 1 "ESP-12E" H 2100 2174 50  0000 C CNN
-F 2 "" H 2100 1500 50  0001 C CNN
-F 3 "http://l0l.org.uk/2014/12/esp8266-modules-hardware-guide-gotta-catch-em-all/" H 2100 1500 50  0001 C CNN
-	1    2100 1500
-	1    0    0    -1
-$EndComp
 Wire Notes Line
 	500  500  500  3300
 Text Notes 700  700  0    50   ~ 0
 ESP8266
-Wire Wire Line
-	1200 1200 850  1200
-Wire Wire Line
-	1200 1400 850  1400
-Wire Wire Line
-	1200 1500 850  1500
-Wire Wire Line
-	850  1600 1200 1600
-Wire Wire Line
-	1200 1700 850  1700
-Wire Wire Line
-	1200 1800 850  1800
 Wire Wire Line
 	850  1900 1200 1900
@@
 GPIO16
 $Comp
-L Device:C C?
+L Device:C C2
 U 1 1 6036934F
 P 3400 2800
-F 0 "C?" H 3515 2846 50  0000 L CNN
+F 0 "C2" H 3515 2846 50  0000 L CNN
 F 1 "100uF" H 3515 2755 50  0000 L CNN
-F 2 "" H 3438 2650 50  0001 C CNN
+F 2 "Capacitor_SMD:C_1206_3216Metric" H 3438 2650 50  0001 C CNN
 F 3 "~" H 3400 2800 50  0001 C CNN
 	1    3400 2800
@@
 $EndComp
 $Comp
-L power:GND #PWR?
+L power:GND #PWR0101
 U 1 1 6036B509
 P 3400 2950
-F 0 "#PWR?" H 3400 2700 50  0001 C CNN
+F 0 "#PWR0101" H 3400 2700 50  0001 C CNN
 F 1 "GND" H 3405 2777 50  0000 C CNN
 F 2 "" H 3400 2950 50  0001 C CNN
@@
 $EndComp
 $Comp
-L power:+3.3V #PWR?
+L power:+3.3V #PWR0102
 U 1 1 6036A9FE
 P 3400 2650
-F 0 "#PWR?" H 3400 2500 50  0001 C CNN
+F 0 "#PWR0102" H 3400 2500 50  0001 C CNN
 F 1 "+3.3V" H 3415 2823 50  0000 C CNN
 F 2 "" H 3400 2650 50  0001 C CNN
@@
 GND
 $Comp
-L power:GND #PWR?
+L power:GND #PWR0103
 U 1 1 604534AE
 P 1350 3050
-F 0 "#PWR?" H 1350 2800 50  0001 C CNN
+F 0 "#PWR0103" H 1350 2800 50  0001 C CNN
 F 1 "GND" H 1355 2877 50  0000 C CNN
 F 2 "" H 1350 3050 50  0001 C CNN
@@
 Vcc
 $Comp
-L power:+3.3V #PWR?
+L power:+3.3V #PWR0104
 U 1 1 6036748F
 P 1000 3000
-F 0 "#PWR?" H 1000 2850 50  0001 C CNN
+F 0 "#PWR0104" H 1000 2850 50  0001 C CNN
 F 1 "+3.3V" H 1015 3173 50  0000 C CNN
 F 2 "" H 1000 3000 50  0001 C CNN
@@
 Power supply
 $Comp
-L power:+12V #PWR?
+L power:+12V #PWR0105
 U 1 1 604956A7
 P 700 3000
-F 0 "#PWR?" H 700 2850 50  0001 C CNN
+F 0 "#PWR0105" H 700 2850 50  0001 C CNN
 F 1 "+12V" H 715 3173 50  0000 C CNN
 F 2 "" H 700 3000 50  0001 C CNN
@@
 	1550 4550 1550 3350
 $Comp
-L Device:R R?
+L Device:R R1
 U 1 1 604A5EDF
 P 4650 1000
-F 0 "R?" V 4750 1000 50  0000 C CNN
-F 1 "12k" V 4534 1000 50  0000 C CNN
-F 2 "" V 4580 1000 50  0001 C CNN
+F 0 "R1" V 4750 1000 50  0000 C CNN
+F 1 "10k" V 4534 1000 50  0000 C CNN
+F 2 "Resistor_SMD:R_0805_2012Metric" V 4580 1000 50  0001 C CNN
 F 3 "~" H 4650 1000 50  0001 C CNN
 	1    4650 1000
@@
 $EndComp
 $Comp
-L Device:R R?
+L Device:R R2
 U 1 1 604A70AC
 P 4650 1350
-F 0 "R?" V 4750 1350 50  0000 C CNN
-F 1 "12k" V 4534 1350 50  0000 C CNN
-F 2 "" V 4580 1350 50  0001 C CNN
+F 0 "R2" V 4750 1350 50  0000 C CNN
+F 1 "10k" V 4534 1350 50  0000 C CNN
+F 2 "Resistor_SMD:R_0805_2012Metric" V 4580 1350 50  0001 C CNN
 F 3 "~" H 4650 1350 50  0001 C CNN
 	1    4650 1350
@@
 $EndComp
 $Comp
-L Device:R R?
+L Device:R R3
 U 1 1 604A9907
 P 4650 1750
-F 0 "R?" V 4750 1750 50  0000 C CNN
-F 1 "12k" V 4534 1750 50  0000 C CNN
-F 2 "" V 4580 1750 50  0001 C CNN
+F 0 "R3" V 4750 1750 50  0000 C CNN
+F 1 "10k" V 4534 1750 50  0000 C CNN
+F 2 "Resistor_SMD:R_0805_2012Metric" V 4580 1750 50  0001 C CNN
 F 3 "~" H 4650 1750 50  0001 C CNN
 	1    4650 1750
@@
 $EndComp
 $Comp
-L Device:R R?
+L Device:R R4
 U 1 1 604A9FC3
 P 4650 2150
-F 0 "R?" V 4750 2150 50  0000 C CNN
-F 1 "12k" V 4534 2150 50  0000 C CNN
-F 2 "" V 4580 2150 50  0001 C CNN
+F 0 "R4" V 4750 2150 50  0000 C CNN
+F 1 "10k" V 4534 2150 50  0000 C CNN
+F 2 "Resistor_SMD:R_0805_2012Metric" V 4580 2150 50  0001 C CNN
 F 3 "~" H 4650 2150 50  0001 C CNN
 	1    4650 2150
@@
 $EndComp
 $Comp
-L Device:R R?
+L Device:R R5
 U 1 1 604AAA90
 P 4650 2850
-F 0 "R?" V 4750 2850 50  0000 C CNN
+F 0 "R5" V 4750 2850 50  0000 C CNN
 F 1 "12k" V 4534 2850 50  0000 C CNN
-F 2 "" V 4580 2850 50  0001 C CNN
+F 2 "Resistor_SMD:R_0805_2012Metric" V 4580 2850 50  0001 C CNN
 F 3 "~" H 4650 2850 50  0001 C CNN
 	1    4650 2850
@@
 	4000 2150 4100 2150
 $Comp
-L Device:C C?
+L Device:C C1
 U 1 1 604B8FCF
 P 4100 2300
-F 0 "C?" H 4215 2346 50  0000 L CNN
+F 0 "C1" H 4215 2346 50  0000 L CNN
 F 1 "100nF" H 4215 2255 50  0000 L CNN
-F 2 "" H 4138 2150 50  0001 C CNN
+F 2 "Capacitor_SMD:C_1206_3216Metric" H 4138 2150 50  0001 C CNN
 F 3 "~" H 4100 2300 50  0001 C CNN
 	1    4100 2300
@@
 	4100 2150 4500 2150
 $Comp
-L power:GND #PWR?
+L power:GND #PWR0106
 U 1 1 604BC712
 P 4100 2450
-F 0 "#PWR?" H 4100 2200 50  0001 C CNN
+F 0 "#PWR0106" H 4100 2200 50  0001 C CNN
 F 1 "GND" H 4105 2277 50  0000 C CNN
 F 2 "" H 4100 2450 50  0001 C CNN
@@
 $EndComp
 $Comp
-L power:GND #PWR?
+L power:GND #PWR0107
 U 1 1 604BD57B
 P 5500 2900
-F 0 "#PWR?" H 5500 2650 50  0001 C CNN
+F 0 "#PWR0107" H 5500 2650 50  0001 C CNN
 F 1 "GND" H 5505 2727 50  0000 C CNN
 F 2 "" H 5500 2900 50  0001 C CNN
@@
 Relay
 $Comp
-L Terminal:Bornera2 U?
+L Terminal:Bornera2 U2
 U 1 1 6045A657
 P 950 3850
-F 0 "U?" H 800 4300 50  0000 L CNN
+F 0 "U2" H 800 4300 50  0000 L CNN
 F 1 "Bornera2" H 800 4200 50  0000 L CNN
-F 2 "" H 950 4200 50  0001 C CNN
+F 2 "Borneras:Bronera_2" H 950 4200 50  0001 C CNN
 F 3 "" H 950 4200 50  0001 C CNN
 	1    950  3850
@@
 Vin
 $Comp
-L power:GND #PWR?
+L power:GND #PWR0108
 U 1 1 6045B47C
 P 600 4050
-F 0 "#PWR?" H 600 3800 50  0001 C CNN
+F 0 "#PWR0108" H 600 3800 50  0001 C CNN
 F 1 "GND" H 605 3877 50  0000 C CNN
 F 2 "" H 600 4050 50  0001 C CNN
@@
 	500  3350 500  4300
 $Comp
-L Terminal:Bornera2 U?
+L Terminal:Bornera2 U3
 U 1 1 60497C27
 P 1250 5050
-F 0 "U?" H 1100 5500 50  0000 L CNN
+F 0 "U3" H 1100 5500 50  0000 L CNN
 F 1 "Bornera2" H 1100 5400 50  0000 L CNN
-F 2 "" H 1250 5400 50  0001 C CNN
+F 2 "Borneras:Bronera_2" H 1250 5400 50  0001 C CNN
 F 3 "" H 1250 5400 50  0001 C CNN
 	1    1250 5050
@@
 Rel_1_out
 $Comp
-L power:GND #PWR?
+L power:GND #PWR0109
 U 1 1 6049AE53
 P 950 5200
-F 0 "#PWR?" H 950 4950 50  0001 C CNN
+F 0 "#PWR0109" H 950 4950 50  0001 C CNN
 F 1 "GND" H 955 5027 50  0000 C CNN
 F 2 "" H 950 5200 50  0001 C CNN
@@
 Text Notes 3050 4950 0    50   ~ 0
 Led indicators
+Wire Wire Line
+	1200 1800 850  1800
+Wire Wire Line
+	1200 1700 850  1700
+Wire Wire Line
+	850  1600 1200 1600
+Wire Wire Line
+	1200 1500 850  1500
+Wire Wire Line
+	1200 1400 850  1400
+Wire Wire Line
+	1200 1200 850  1200
+$Comp
+L ESP_8366_CUSTOM:ESP-12E U1
+U 1 1 60363FD8
+P 2100 1500
+F 0 "U1" H 2100 2265 50  0000 C CNN
+F 1 "ESP-12E" H 2100 2174 50  0000 C CNN
+F 2 "RF_Module:ESP-12E" H 2100 1500 50  0001 C CNN
+F 3 "http://l0l.org.uk/2014/12/esp8266-modules-hardware-guide-gotta-catch-em-all/" H 2100 1500 50  0001 C CNN
+	1    2100 1500
+	1    0    0    -1
+$EndComp
 $EndSCHEMATC

Commit message: .
Parts:
- U1: footprint RF_Module:ESP-12E -> Esp8266_Module:C_WiFiModule
Changed lines of the file:
@@
 F 0 "U1" H 2100 2265 50  0000 C CNN
 F 1 "ESP-12E" H 2100 2174 50  0000 C CNN
-F 2 "RF_Module:ESP-12E" H 2100 1500 50  0001 C CNN
+F 2 "Esp8266_Module:C_WiFiModule" H 2100 1500 50  0001 C CNN
 F 3 "http://l0l.org.uk/2014/12/esp8266-modules-hardware-guide-gotta-catch-em-all/" H 2100 1500 50  0001 C CNN
 	1    2100 1500
