File: HW_design/Access_control/Relay_output.sch (KiCad schematic (older format))
At the start: 4 parts

Commit message: pcb design
Parts:
- D1: renamed from D?; footprint (none) -> SMD_DIODE_3.20mmx8.13mm:SMD_DIODE_3.2mmx8.13mm
- R6: renamed from R?; footprint (none) -> Resistor_SMD:R_0805_2012Metric
- RELAY1: renamed from RELAY?; footprint (none) -> Relay_5pin:Relay
- gave numbers to parts that had none: 1
Connections:
- no-connect marks 0 -> 1
Changed lines of the file:
@@
 $EndDescr
 $Comp
-L Relay_5_pin:JQC-3FF RELAY?
+L Relay_5_pin:JQC-3FF RELAY1
 U 1 1 6046C01D
 P 3100 1250
-F 0 "RELAY?" H 3528 1296 50  0000 L CNN
+F 0 "RELAY1" H 3528 1296 50  0000 L CNN
 F 1 "JQC-3FF" H 3528 1205 50  0000 L CNN
-F 2 "" H 3700 1200 50  0001 C CNN
+F 2 "Relay_5pin:Relay" H 3700 1200 50  0001 C CNN
 F 3 "" H 3700 1200 50  0001 C CNN
 	1    3100 1250
@@
 $EndComp
 $Comp
-L Device:D_Schottky_ALT D?
+L Device:D_Schottky_ALT D1
 U 1 1 6046DDCE
 P 2550 1250
-F 0 "D?" V 2450 1050 50  0000 L CNN
+F 0 "D1" V 2450 1050 50  0000 L CNN
 F 1 "D_Schottky_ALT" V 2650 550 50  0000 L CNN
-F 2 "" H 2550 1250 50  0001 C CNN
+F 2 "SMD_DIODE_3.20mmx8.13mm:SMD_DIODE_3.2mmx8.13mm" H 2550 1250 50  0001 C CNN
 F 3 "~" H 2550 1250 50  0001 C CNN
 	1    2550 1250
@@
 	2850 1650 2850 1850
 $Comp
-L power:GND #PWR?
+L power:GND #PWR0113
 U 1 1 60472962
 P 2850 2350
-F 0 "#PWR?" H 2850 2100 50  0001 C CNN
+F 0 "#PWR0113" H 2850 2100 50  0001 C CNN
 F 1 "GND" H 2855 2177 50  0000 C CNN
 F 2 "" H 2850 2350 50  0001 C CNN
@@
 	2850 2250 2850 2350
 $Comp
-L Device:R R?
+L Device:R R6
 U 1 1 604735CF
 P 2250 2050
-F 0 "R?" V 2043 2050 50  0000 C CNN
+F 0 "R6" V 2043 2050 50  0000 C CNN
 F 1 "2.2k" V 2134 2050 50  0000 C CNN
-F 2 "" V 2180 2050 50  0001 C CNN
+F 2 "Resistor_SMD:R_0805_2012Metric" V 2180 2050 50  0001 C CNN
 F 3 "~" H 2250 2050 50  0001 C CNN
 	1    2250 2050
@@
 Rel_1_out
 $Comp
-L Transistor_BJT:MMBT3904 Q?
+L Transistor_BJT:MMBT3904 Q1
 U 1 1 604C5FC3
 P 2750 2050
-F 0 "Q?" H 2941 2096 50  0000 L CNN
+F 0 "Q1" H 2941 2096 50  0000 L CNN
 F 1 "MMBT3904" H 2941 2005 50  0000 L CNN
 F 2 "Package_TO_SOT_SMD:SOT-23" H 2950 1975 50  0001 L CIN
@@
 	1    0    0    -1
 $EndComp
+NoConn ~ 3300 900
 $EndSCHEMATC

Commit message: .
Parts:
- D1: footprint SMD_DIODE_3.20mmx8.13mm:SMD_DIODE_3.2mmx8.13mm -> SMD_DIODE_3.20mmx8.13mm:SMD_DIODE_4.6mmx2.90
Changed lines of the file:
@@
 F 0 "D1" V 2450 1050 50  0000 L CNN
 F 1 "D_Schottky_ALT" V 2650 550 50  0000 L CNN
-F 2 "SMD_DIODE_3.20mmx8.13mm:SMD_DIODE_3.2mmx8.13mm" H 2550 1250 50  0001 C CNN
+F 2 "SMD_DIODE_3.20mmx8.13mm:SMD_DIODE_4.6mmx2.90" H 2550 1250 50  0001 C CNN
 F 3 "~" H 2550 1250 50  0001 C CNN
 	1    2550 1250
